File: hardware/smart-ballot-box/sbb-shield.brd (EAGLE design)
At the start: 68.6 x 53.3 mm, 56 parts, among them IC1 DS1338-33, IC2 LM393D, IC4 DRV8871DDA, U1 MICROSD

Commit message: schematic coming together.
Parts:
- removed C2, C3: 1uf, rcl:C0603K
- removed C8: 10uf, resistor:C1206K
- removed R8: 220, resistor:R0603
- removed R9: 360, resistor:R0603
- removed U4: (no value), SparkFun-IC-Power:SOT223
- added C12, C9: .1uf, rcl:C0603K
- added C13: .1uf, adafruit:C0603K
- added R22, R23: 10k, adafruit:R0603
- added R24, R25: 33k, adafruit:R0603
- C6: value (none) -> 22uF / 63V
- C7: value (none) -> .1uf/50V
- R10: value 220 -> 500
- R11: value 360 -> 220
- TM1, TM2: value (none) -> 10k
- moved R10 174.0 mm to (35.2, 36.8), turned to 270 degrees
- moved U2 172.9 mm to (38.1, 43.2)
- moved R11 172.2 mm to (33.0, 36.8), turned to 90 degrees
- moved C10 172.0 mm to (37.1, 36.8), turned to 90 degrees
- moved C11 161.6 mm to (39.0, 35.6), turned to 90 degrees
- moved J1 144.5 mm to (12.4, 49.8), turned to 180 degrees
- moved T3 124.5 mm to (55.9, 44.5), turned to 270 degrees
- moved R12 117.6 mm to (53.3, 44.5), turned to 270 degrees
- moved R13 117.6 mm to (58.4, 44.5), turned to 270 degrees
- moved R15 106.7 mm to (41.5, 28.4), turned to 270 degrees
- moved R14 106.4 mm to (36.1, 28.3), turned to 270 degrees
- moved SPOIL_BTN1 101.8 mm to (55.9, 33.0), turned to 90 degrees
- moved T4 100.9 mm to (38.7, 28.4), turned to 270 degrees
- moved R6 98.3 mm to (47.0, 45.7)
- moved IC1 97.7 mm to (4.83, 3.56), turned to 90 degrees
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Connections:
- removed net N$11: R8.1, R9.2, U4.1
- removed net N$17: C4.1, IC2.1, R17.1
- removed net N$18: C5.1, IC2.7, R16.1
- removed net N$19: SPOIL_BTN1.1
- removed net N$20: IC2.5, PAPER_IN.2
- removed net N$21: IC2.3, PAPER_OUT.2
- removed net N$25: R13.2, T3.3
- removed net N$31: CAST_BTN1.1
- removed net N$32: R15.2, T4.3
- removed net N$4: U$2.A0
- removed net N$5: U$2.A1
- removed net N$6: U$2.A2
- removed net N$7: U$2.A3
- removed net SCL1: PMOD1.7
- removed net SDA1: PMOD1.5
- new net GPIOX.0: C4.1, IC2.1, PMOD1.5, R17.1, U$2.A3
- new net GPIOX.1: C5.1, IC2.7, PMOD1.7, R16.1, U$2.A2
- new net N$13: IC2.2, PAPER_OUT.2
- new net N$15: IC2.6, PAPER_IN.2
- new net SCAN_DIN: R21.1, SCANNER1.3, T6.1, U$2.D1
- new net SCAN_DOUT: R19.1, SCANNER1.2, T5.1, U$2.D0
- net +12V: no longer C3.2, U2.3, U4.3
- net +3V3: now also C13.1, PMOD1.11, PMOD1.12, PMOD2.11, PMOD2.12, R24.2, R25.2, TM1.1, TM2.1, U2.3; no longer C2.2, C8.2, R8.2, U4.2, U4.4
- net GND: now also C12.2, C13.2, C9.2, R22.1, R23.1, TM1.3, TM2.3; no longer C2.1, C3.1, C8.1, R9.1
- net GPIO1.0: now also C12.1, R23.2, SPOIL_BTN1.1, U$2.D5
- net GPIO1.1: now also R13.2, T3.3, U$2.D4
- net GPIO1.2: now also C9.1, CAST_BTN1.1, R22.2, U$2.D3
- net GPIO1.3: now also R15.2, T4.3, U$2.D2
- net GPIO2.0: now also U$2.D7
- net GPIO2.1: now also U$2.D6
- net N$1: now also IC2.5, R24.1, TM2.2; no longer R21.1, SCANNER1.3, T6.1
- net N$2: now also IC2.3, R25.1, TM1.2; no longer R19.1, SCANNER1.2, T5.1
- net UART1_RX: no longer U$2.D0
- net UART1_TX: no longer U$2.D1
Routing:
- net +3V3: track 0.00 -> 276.1 mm, vias 0 -> 2
- net SCK: track 0.00 -> 110.6 mm, vias 0 -> 1
- net MOSI: track 0.00 -> 108.6 mm, vias 0 -> 1
- net MISO: track 0.00 -> 107.4 mm, vias 0 -> 1
- net SS: track 0.00 -> 105.2 mm, vias 0 -> 1
- net GPIO2.0: track 0.00 -> 98.8 mm, vias 0 -> 2
- net GPIO2.1: track 0.00 -> 93.6 mm, vias 0 -> 2
- net SDA0: track 0.00 -> 90.6 mm, vias 0 -> 1
- net SCL0: track 0.00 -> 83.5 mm, vias 0 -> 2
- net GPIO1.3: track 0.00 -> 55.4 mm, vias 0 -> 2
- net GPIOX.0: track 0.00 -> 53.1 mm, vias 0 -> 1
- net GPIO1.0: track 0.00 -> 48.0 mm
- net SCAN_DOUT: track 0.00 -> 47.3 mm, vias 0 -> 3
- net SCAN_DIN: track 0.00 -> 44.7 mm
- net GPIOX.1: track 0.00 -> 44.5 mm, vias 0 -> 1
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- added copper zone on layer 15, net CUTOUT
- added copper zone on layer 2, net CUTOUT
- added copper zone on layer 1, net GND
- added copper zone on layer 15, net GND
- added copper zone on layer 16, net GND
- added copper zone on layer 2, net GND
Other:
- board text added: "+"
- board text added: "-"
- board text added: "Smart Ballot Box Shield v0"

Commit message: revision 2
Parts:
- removed BATT1: LR44, bitsetters:LR44
- removed Q2: (no value), adafruit (DESKTOP-MKQ6VR9's conflicted copy 2019-02-08):TC26H
- added G1: 10MM_SM_COIN_CELL_CLIP, battery:10MM_SM_COIN_CELL_CLIP
- added LED1: (no value), adafruit:CHIP-LED0603
- added Q1: 32.768khz, adafruit (DESKTOP-MKQ6VR9's conflicted copy 2019-02-08):TC26H
- added R26: 500, resistor:R0603
- added R8: 68R, adafruit:R0603
- added R9: 100R, adafruit:R0603
- added Y1: 32.768khz, SamacSys_Parts:ABS07AIG32768KHZ71T
- C1: value (none) -> .1uf
- R1, R3: value (none) -> 2.2k
- R12, R14: value 1k -> 68R
- R2, R4, R5, R7: value (none) -> 10k
- T3, T4, T5, T6: value (none) -> PMV65UNEAR
- moved C12 1.45 mm to (60.7, 39.4)
- moved R23 1.30 mm to (60.6, 41.3)
- moved R17 1.14 mm to (38.0, 8.97)
- moved R13 0.97 mm to (59.0, 45.2)
- moved R25 0.93 mm to (41.7, 7.62)
- moved R12 0.86 mm to (53.2, 45.3)
- moved T3 0.77 mm to (56.0, 45.2)
- moved TM1 0.72 mm to (35.0, 9.02)
- flipped PMOD0 to the bottom
- flipped PMOD1 to the bottom
- renumbered CAST_BTN1 to CAST_BTN, MOTOR1 to MOTOR, PMOD2 to PMOD0, SCANNER1 to SCANNER, SPOIL_BTN1 to SPOIL_BTN
Connections:
- new net N$4: LED1.C, R26.1
- new net N$5: PAPER_OUT.3, R25.2, R8.2, R9.1, TM1.1
- net +3V3: now also LED1.A, R9.2; no longer PAPER_OUT.3, R25.2, TM1.1
- net GND: now also G1.-, R26.2, R8.1; no longer BATT1.N1, BATT1.N2
- net N$3: now also Q1.1, Y1.2; no longer Q2.2
- net N$8: now also Q1.2, Y1.1; no longer Q2.1
- net N$9: now also G1.+@1, G1.+@2; no longer BATT1.P1
Routing:
- net +3V3: track 276.1 -> 245.8 mm, vias 2 -> 7
- net N$5: track 0.00 -> 25.1 mm
- net N$9: track 20.3 -> 27.8 mm
- net UART1_TX: track 34.4 -> 39.0 mm
- net GPIO1.2: track 40.9 -> 37.2 mm
- net UART1_RX: track 42.9 -> 46.3 mm
- net GPIO1.1: track 37.1 -> 40.4 mm
- net N$3: track 2.62 -> 5.80 mm
- net SCK: track 110.6 -> 107.5 mm
- net N$8: track 3.15 -> 6.16 mm
- net MOSI: track 108.6 -> 105.6 mm
- net GPIOX.0: track 53.1 -> 50.1 mm
- net MISO: track 107.4 -> 104.5 mm
- net SS: track 105.2 -> 102.4 mm
- net SDA0: track 90.6 -> 93.4 mm
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Other:
- board text added: "POWER"
- board text added: "Smart Ballot Box Shield R2"
- board text removed: "Smart Ballot Box Shield v0"
