File: hardware/smart-ballot-box/sbb-shield.sch (EAGLE design)
At the start: 56 parts, among them IC1 DS1338-33, IC2 LM393D, IC4 DRV8871DDA, U1 MICROSD

Commit message: schematic coming together.
Parts:
- removed C2, C3: 1uf, rcl:C-USC0603K
- removed C8: 10uf, resistor:C-USC1206K
- removed R8: 220, resistor:R-US_R0603
- removed R9: 360, resistor:R-US_R0603
- removed U4: (no value), SparkFun-IC-Power:V_REG_LM1117SOT223
- added C12, C9: .1uf, rcl:C-USC0603K
- added C13: .1uf, adafruit:C-USC0603K
- added R22, R23: 10k, adafruit:R-US_R0603
- added R24, R25: 33k, adafruit:R-US_R0603
- C6: value (none) -> 22uF / 63V
- C7: value (none) -> .1uf/50V
- R10: value 220 -> 500
- R11: value 360 -> 220
- TM1, TM2: value (none) -> 10k
Connections:
- removed net N$11: R8.1, R9.2, U4.ADJ
- removed net N$17: C4.1, IC2A.OUT, R17.1
- removed net N$18: C5.1, IC2B.OUT, R16.1
- removed net N$19: SPOIL_BTN1.1
- removed net N$20: IC2B.+IN, PAPER_IN.2
- removed net N$21: IC2A.+IN, PAPER_OUT.2
- removed net N$25: R13.2, T3.G
- removed net N$31: CAST_BTN1.1
- removed net N$32: R15.2, T4.G
- removed net N$4: U$2.A0
- removed net N$5: U$2.A1
- removed net N$6: U$2.A2
- removed net N$7: U$2.A3
- removed net SCL1: PMOD1.7
- removed net SDA1: PMOD1.5
- new net GPIOX.0: C4.1, IC2A.OUT, PMOD1.5, R17.1, U$2.A3
- new net GPIOX.1: C5.1, IC2B.OUT, PMOD1.7, R16.1, U$2.A2
- new net N$13: IC2A.-IN, PAPER_OUT.2
- new net N$15: IC2B.-IN, PAPER_IN.2
- new net SCAN_DIN: R21.1, SCANNER1.3, T6.D, U$2.D1
- new net SCAN_DOUT: R19.1, SCANNER1.2, T5.D, U$2.D0
- net +12V: no longer C3.2, U2.IN, U4.IN
- net +3V3: now also C13.1, PMOD1.11, PMOD1.12, PMOD2.11, PMOD2.12, R24.2, R25.2, TM1.A, TM2.A, U2.IN; no longer C2.2, C8.2, R8.2, U4.OUT, U4.OUT@1
- net GND: now also C12.2, C13.2, C9.2, R22.1, R23.1, TM1.E, TM2.E; no longer C2.1, C3.1, C8.1, R9.1
- net GPIO1.0: now also C12.1, R23.2, SPOIL_BTN1.1, U$2.D5
- net GPIO1.1: now also R13.2, T3.G, U$2.D4
- net GPIO1.2: now also C9.1, CAST_BTN1.1, R22.2, U$2.D3
- net GPIO1.3: now also R15.2, T4.G, U$2.D2
- net GPIO2.0: now also U$2.D7
- net GPIO2.1: now also U$2.D6
- net N$1: now also IC2B.+IN, R24.1, TM2.S; no longer R21.1, SCANNER1.3, T6.D
- net N$2: now also IC2A.+IN, R25.1, TM1.S; no longer R19.1, SCANNER1.2, T5.D
- net UART1_RX: no longer U$2.D0
- net UART1_TX: no longer U$2.D1
Other:
- note added: "1"
- note added: "1.8v logic for GFE"
- note added: "2A Peak (Short duration!) 45V Max PWM: 0-100kHz"
- note added: "500ma MAX"
- note added: "Button SPST, NC: P1: BUTTON GPIO, active high P2: +3.3V to button LED: P3: GPIO, high = ON P4: +3.3V to LED"
- note added: "Connects to Sparkfun LCD-14073 via I2C"
- note added: "Connects to Waveshare 1D/2D barcode reader module UPC 614961952195"
- note added: "DS1338 is a 3.3v part compatible with DS1307"
- note added: "I2C Pullups"
- note added: "LCD & RTC"
- note added: "MicroSD Card"
- note added: "Motor"
- note added: "PAPER_IN connects to Sparkfun RedBot Sensor - Line Follower PN: SEN-11769"
- note added: "PAPER_OUT connects to optical endstop switch common to 3D printers. Amazon ASIN B077X8XL56"
- note added: "Paper Present Active Low"
- note added: "Unbuffered 3.3v"
- note removed: "Fixed 3V3 use R9=0R, R8=NP"
- note removed: "LED"
- note removed: "NEED GPIO"
- moved on the sheet: C10, C11, C4, C5, C6, CAST_BTN1, IC2A, IC2B, J1, MOTOR1, PAPER_IN, PMOD2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

Commit message: revision 2
Parts:
- removed BATT1: LR44, bitsetters:LR44
- removed Q2: (no value), adafruit (DESKTOP-MKQ6VR9's conflicted copy 2019-02-08):CRYSTALTC26H
- added G1: 10MM_SM_COIN_CELL_CLIP, battery:10MM_SM_COIN_CELL_CLIP
- added LED1: (no value), adafruit:LEDCHIP-LED0603
- added Q1: 32.768khz, adafruit (DESKTOP-MKQ6VR9's conflicted copy 2019-02-08):CRYSTALTC26H
- added R26: 500, resistor:R-US_R0603
- added R8: 68R, adafruit:R-US_R0603
- added R9: 100R, adafruit:R-US_R0603
- added Y1: 32.768khz, SamacSys_Parts:ABS07W-32.768KHZ-D-1-T
- C1: value (none) -> .1uf
- R1, R3: value (none) -> 2.2k
- R12, R14: value 1k -> 68R
- R2, R4, R5, R7: value (none) -> 10k
- T3, T4, T5, T6: value (none) -> PMV65UNEAR
- renumbered CAST_BTN1 to CAST_BTN, MOTOR1 to MOTOR, PMOD2 to PMOD0, SCANNER1 to SCANNER, SPOIL_BTN1 to SPOIL_BTN
Connections:
- new net N$4: LED1.C, R26.1
- new net N$5: PAPER_OUT.3, R25.2, R8.2, R9.1, TM1.A
- net +3V3: now also LED1.A, R9.2; no longer PAPER_OUT.3, R25.2, TM1.A
- net GND: now also G1.-, R26.2, R8.1; no longer BATT1.NEG
- net N$3: now also Q1.1, Y1.2; no longer Q2.2
- net N$8: now also Q1.2, Y1.1; no longer Q2.1
- net N$9: now also G1.+; no longer BATT1.POS
Other:
- note added: "1. 5/31 R1 - Initial Release 2. 6/9 R2 * Clearer Soldermask labels for connectors * Fixed mirroed PMOD connectors * Changed LED resistor value from 1k to 68R * Added additional footprint for RTC crystal to accomidate SMD options. * Fixed battery clip so battery can be inserted correctly. Previously was backward. * Changed from 1.5V LR44 to 3V CR927 * Added optional resistor divider to accomidate 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"
- note added: "2"
- note added: "Fixed 1V8 use R11=0R, R10=NP"
- note added: "Revision History"
- note removed: "1"
- note removed: "Fixed 1V8 use R9=0R, R8=NP"
